File: board/TD-M5037/TD-M5037.kicad_pcb (KiCad board)
At the start: 2 copper layers, 50 x 37 mm, 25 parts, among them J1 Pin 1x5, J4 Pin 1x6, J5 PowerPad, J8 PowerPad, U2 DS1307, U3 ATmega328PB-QFP, Y1 16MHz, Y2 32.768KHz

Commit message: Cleanup 3d prints
Other:
- board text added: "Not Needed Unless you want UART"
Changed lines of the file:
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@@
         (effects (font (size 1 1) (thickness 0.1)) (justify mirror))
     )
-    (fp_text value "PowerPad" (at 0 -0.031 unlocked) (layer "B.Fab")
+    (fp_text value "PowerPad" (at 0 -0.031 unlocked) (layer "B.Fab") hide
         (effects (font (size 1 1) (thickness 0.15)) (justify mirror))
     )
@@
         (effects (font (size 1 1) (thickness 0.1)) (justify mirror))
     )
-    (fp_text value "PowerPad" (at 0 -0.031 unlocked) (layer "B.Fab")
+    (fp_text value "PowerPad" (at 0 -0.031 unlocked) (layer "B.Fab") hide
         (effects (font (size 1 1) (thickness 0.15)) (justify mirror))
     )
@@
     (effects (font (size 1 1) (thickness 0.15)) (justify bottom mirror))
   )
-  (gr_text "Not Needed" (at 69.85 76.835 90) (layer "B.Fab")
-    (effects (font (size 1 1) (thickness 0.15)) (justify left bottom mirror))
+  (gr_text "Not Needed\nUnless you want UART" (at 69.85 76.835 90) (layer "B.Fab")
+    (effects (font (size 1 1) (thickness 0.15)) (justify bottom mirror))
   )
   (gr_text "TokeiDigital\nMovement 5037 REV.A" (at 104.775 92.71) (layer "F.Fab")

Commit message: Prepare for sale
Parts:
- C4: value 100nF -> 3x100nF
- D3: value 1N5817 -> 2x1N5817
- renumbered locked to BT1, locked to J6, locked to J7
Other:
- board text added: "+5V"
- board text added: "GND"
- board text added: "ICSP"
- board text added: "Movement 5037 REV.A"
- board text added: "Not Needed ICSP"
- board text added: "Not Needed Unless you want UART If assembled, assemble on this side"
- board text added: "Pin 1x6"
- board text added: "UART"
- board text removed: "Not Needed"
- board text removed: "Not Needed Unless you want UART"
- board text removed: "locked"
