File: board/TD-TOE01/power.kicad_sch (KiCad schematic)
At the start: 4 parts, among them J5 PowerPad, J6 PowerPad

Commit message: OET schematic
Parts:
- added D4: LED1206, LED_SMD:LED_1206_3216Metric, symbol TokeiDigital:LED1206
- added R8: 1K, TokeiDigital:R_0805, symbol Device:R
- added S1: SWITCH-DPDT, symbol TokeiDigital:SWITCH-DPDT
- added U12: ~, symbol TokeiDigital:LipoCharger
- J5: value PowerPad -> BAT+
- J6: value PowerPad -> BAT-
Connections:
- net +5V: now also R8.1
- net GND: now also D4.1 (K), U12.4 (OUT-); no longer J6.1
- net at D3.2 (A): now also S1.5; no longer J5.1
- new net: J6.1, U12.3 (BAT-)
- new net: D4.2 (A), R8.2
- new net: S1.6, U12.1 (OUT+)
- new net: J5.1, U12.2 (BAT+)
- no-connect marks 0 -> 7
Other:
- moved on the sheet: C8, D3, J5
