File: board/TD-TOE01/TD-TOE01.kicad_pcb (KiCad board)
At the start: 2 copper layers, 0 parts

Commit message: OET First steps
Parts:
- added BT1: CR3032 Holder, TokeiDigital:CR2032 Holder, F.Cu at (37.0, 68.4)
- added C1: 100nF, TokeiDigital:C_0805, F.Cu at (49.3, 38.6)
- added C2: 100nF, TokeiDigital:C_0805, F.Cu at (73.4, 57.6)
- added C3: 100nF, TokeiDigital:C_0805, F.Cu at (73.4, 60.6)
- added C4: 100nF, TokeiDigital:C_0805, F.Cu at (73.4, 63.7)
- added C5: 22p, TokeiDigital:C_0805, F.Cu at (73.4, 66.7)
- added C6: 22p, TokeiDigital:C_0805, F.Cu at (73.4, 69.7)
- added C7: 100nF, TokeiDigital:C_0805, F.Cu at (73.4, 72.7)
- added C8: 10uF, TokeiDigital:C_1206, F.Cu at (80.0, 93.6)
- added C9: 100nF, TokeiDigital:C_0805, F.Cu at (44.9, 82.2)
- added D1: 1N5817, TokeiDigital:D_2010, F.Cu at (89.2, 79.2)
- added D2: 1N5817, TokeiDigital:D_2010, F.Cu at (89.2, 83.5)
- added D3: 1N5817, TokeiDigital:D_2010, F.Cu at (80.9, 89.8)
- added J1: Pin 1x6, TokeiDigital:PIN 1x06, F.Cu at (78.3, 58.5)
- added J2: AVR-ISP, TokeiDigital:PIN 2x03, F.Cu at (78.3, 75.9)
- added J3: Pin 1x5, TokeiDigital:PIN 1x05, F.Cu at (87.7, 58.5)
- added J4: Pin 1x6, TokeiDigital:PIN 1x06, F.Cu at (83.0, 58.5)
- added J5: PowerPad, TokeiDigital:Power Pin, F.Cu at (74.0, 90.6)
- added J6: PowerPad, TokeiDigital:Power Pin, F.Cu at (74.0, 96.6)
- added R1: 10K, TokeiDigital:R_0805, F.Cu at (49.3, 41.6)
- added R2: 10K, TokeiDigital:R_0805, F.Cu at (73.4, 75.7)
- added R3: 10K, TokeiDigital:R_0805, F.Cu at (73.4, 78.6)
- added R4: 10K, TokeiDigital:R_0805, F.Cu at (73.4, 81.6)
- added U1: MAX7221xWG, Package_SO:SOIC-24W_7.5x15.4mm_P1.27mm, F.Cu at (40.5, 45.7)
- added U2: Sx39-1xxxxx, TokeiDigital:3191AS, F.Cu at (36.2, 24.7)
- added U3: Sx39-1xxxxx, TokeiDigital:3191AS, F.Cu at (48.0, 24.7)
- added U4: Sx39-1xxxxx, TokeiDigital:3191AS, F.Cu at (59.9, 24.7)
- added U5: Sx39-1xxxxx, TokeiDigital:3191AS, F.Cu at (71.7, 24.7)
- added U6: Sx39-1xxxxx, TokeiDigital:3191AS, F.Cu at (83.5, 24.7)
- added U7: Sx39-1xxxxx, TokeiDigital:3191AS, F.Cu at (95.3, 24.7)
- added U8: ATmega328PB-QFP, TokeiDigital:TQFP-32, F.Cu at (95.8, 62.0)
- added U9: DS1307, TokeiDigital:SOIC-8, F.Cu at (38.2, 83.9)
- added Y1: 16MHz, TokeiDigital:Crystal Vertical, F.Cu at (89.3, 73.7)
- added Y2: 32.768KHz, TokeiDigital:Crystal Horizontal, F.Cu at (65.8, 57.5)
Other:
- board text removed: "Movement 5037 REV.A"

Commit message: OET
Parts:
- added C1: 10uF, TokeiDigital:C_1206, B.Cu at (-107.2, 46.0)
- added C11: 100nF, TokeiDigital:C_1206, B.Cu at (-97.8, 85.5)
- added C12: 100nF, TokeiDigital:C_1206, B.Cu at (-97.8, 89.5)
- added C13: 10nF, TokeiDigital:C_1206, B.Cu at (-97.8, 93.5)
- added C14: 1uF, TokeiDigital:C_1206, B.Cu at (-97.8, 97.6)
- added C15: 1uF, TokeiDigital:C_1206, B.Cu at (-97.8, 101.7)
- added C3: 100nF, TokeiDigital:C_1206, B.Cu at (-82.9, 102.5)
- added D1: 1N5817, TokeiDigital:D_2010, B.Cu at (-101.3, 41.8)
- added D10: LED1206, LED_SMD:LED_1206_3216Metric, F.Cu at (179.4, 61.7)
- added D11: LED1206, LED_SMD:LED_1206_3216Metric, F.Cu at (186.5, 61.7)
- added D12: LED1206, LED_SMD:LED_1206_3216Metric, F.Cu at (136.8, 69.8)
- added D13: LED1206, LED_SMD:LED_1206_3216Metric, F.Cu at (143.9, 69.8)
- added D14: LED1206, LED_SMD:LED_1206_3216Metric, F.Cu at (151.0, 69.8)
- added D15: LED1206, LED_SMD:LED_1206_3216Metric, F.Cu at (158.1, 69.8)
- added D16: LED1206, LED_SMD:LED_1206_3216Metric, F.Cu at (165.2, 69.8)
- added D17: LED1206, LED_SMD:LED_1206_3216Metric, F.Cu at (172.3, 69.8)
- added D18: LED1206, LED_SMD:LED_1206_3216Metric, F.Cu at (179.4, 69.8)
- added D19: LED1206, LED_SMD:LED_1206_3216Metric, F.Cu at (186.5, 69.8)
- added D2: LED1206, LED_SMD:LED_1206_3216Metric, B.Cu at (-108.3, 49.7)
- added D20: LED1206, LED_SMD:LED_1206_3216Metric, F.Cu at (136.8, 78.0)
- added D21: LED1206, LED_SMD:LED_1206_3216Metric, F.Cu at (143.9, 78.0)
- added D22: LED1206, LED_SMD:LED_1206_3216Metric, F.Cu at (151.0, 78.0)
- added D23: LED1206, LED_SMD:LED_1206_3216Metric, F.Cu at (158.1, 78.0)
- added D24: LED1206, LED_SMD:LED_1206_3216Metric, F.Cu at (165.2, 78.0)
- added D25: LED1206, LED_SMD:LED_1206_3216Metric, F.Cu at (172.3, 78.0)
- added D26: LED1206, LED_SMD:LED_1206_3216Metric, F.Cu at (179.4, 78.0)
- added D27: LED1206, LED_SMD:LED_1206_3216Metric, F.Cu at (186.5, 78.0)
- added D28: LED1206, LED_SMD:LED_1206_3216Metric, F.Cu at (136.8, 86.2)
- added D29: LED1206, LED_SMD:LED_1206_3216Metric, F.Cu at (143.9, 86.2)
- added D3: LED1206, LED_SMD:LED_1206_3216Metric, F.Cu at (-43.2, 148.7)
- added D30: LED1206, LED_SMD:LED_1206_3216Metric, F.Cu at (151.0, 86.2)
- added D31: LED1206, LED_SMD:LED_1206_3216Metric, F.Cu at (158.1, 86.2)
- added D32: LED1206, LED_SMD:LED_1206_3216Metric, F.Cu at (165.2, 86.2)
- added D33: LED1206, LED_SMD:LED_1206_3216Metric, F.Cu at (172.3, 86.2)
- added D34: LED1206, LED_SMD:LED_1206_3216Metric, F.Cu at (179.4, 86.2)
- added D35: LED1206, LED_SMD:LED_1206_3216Metric, F.Cu at (186.5, 86.2)
- added D36: LED1206, LED_SMD:LED_1206_3216Metric, F.Cu at (170.5, 51.0)
- added D37: LED1206, LED_SMD:LED_1206_3216Metric, F.Cu at (194.0, 51.0)
- added D38: LED1206, LED_SMD:LED_1206_3216Metric, F.Cu at (-38.2, 164.2)
- added D39: LED1206, LED_SMD:LED_1206_3216Metric, F.Cu at (-38.2, 167.6)
- added D4: LED1206, LED_SMD:LED_1206_3216Metric, F.Cu at (136.8, 61.7)
- added D40: LED1206, LED_SMD:LED_1206_3216Metric, F.Cu at (-38.2, 170.9)
- added D41: LED1206, LED_SMD:LED_1206_3216Metric, F.Cu at (-38.2, 174.3)
- added D42: LED1206, LED_SMD:LED_1206_3216Metric, F.Cu at (-38.2, 177.7)
- added D43: LED1206, LED_SMD:LED_1206_3216Metric, F.Cu at (-38.2, 181.1)
- added D44: LED1206, LED_SMD:LED_1206_3216Metric, F.Cu at (-38.2, 184.5)
- added D45: LED1206, LED_SMD:LED_1206_3216Metric, F.Cu at (-38.2, 187.9)
- added D46: LED1206, LED_SMD:LED_1206_3216Metric, F.Cu at (-38.2, 191.3)
- added D47: LED1206, LED_SMD:LED_1206_3216Metric, F.Cu at (-32.5, 157.4)
- added D48: LED1206, LED_SMD:LED_1206_3216Metric, F.Cu at (-32.5, 160.8)
- added D49: LED1206, LED_SMD:LED_1206_3216Metric, F.Cu at (-32.5, 164.2)
- added D5: LED1206, LED_SMD:LED_1206_3216Metric, F.Cu at (143.9, 61.7)
- added D50: LED1206, LED_SMD:LED_1206_3216Metric, F.Cu at (-32.5, 167.6)
- added D51: LED1206, LED_SMD:LED_1206_3216Metric, F.Cu at (-32.5, 170.9)
- added D52: LED1206, LED_SMD:LED_1206_3216Metric, F.Cu at (-32.5, 174.3)
- added D53: LED1206, LED_SMD:LED_1206_3216Metric, F.Cu at (-32.5, 177.7)
- added D54: LED1206, LED_SMD:LED_1206_3216Metric, F.Cu at (-32.5, 181.1)
- added D55: LED1206, LED_SMD:LED_1206_3216Metric, F.Cu at (-32.5, 184.5)
- added D56: LED1206, LED_SMD:LED_1206_3216Metric, F.Cu at (-32.5, 187.9)
- added D57: LED1206, LED_SMD:LED_1206_3216Metric, F.Cu at (-32.5, 191.3)
- added D58: LED1206, LED_SMD:LED_1206_3216Metric, F.Cu at (-26.9, 157.4)
- added D59: LED1206, LED_SMD:LED_1206_3216Metric, F.Cu at (-26.9, 160.8)
- added D6: LED1206, LED_SMD:LED_1206_3216Metric, F.Cu at (151.0, 61.7)
- added D60: LED1206, LED_SMD:LED_1206_3216Metric, F.Cu at (-26.9, 164.2)
- added D61: LED1206, LED_SMD:LED_1206_3216Metric, F.Cu at (-26.9, 167.6)
- added D62: LED1206, LED_SMD:LED_1206_3216Metric, F.Cu at (-26.9, 170.9)
- added D63: LED1206, LED_SMD:LED_1206_3216Metric, F.Cu at (-26.9, 174.3)
- added D64: LED1206, LED_SMD:LED_1206_3216Metric, F.Cu at (-26.9, 177.7)
- added D65: LED1206, LED_SMD:LED_1206_3216Metric, F.Cu at (-26.9, 181.1)
- added D66: LED1206, LED_SMD:LED_1206_3216Metric, F.Cu at (-26.9, 184.5)
- added D7: LED1206, LED_SMD:LED_1206_3216Metric, F.Cu at (158.1, 61.7)
- added D8: LED1206, LED_SMD:LED_1206_3216Metric, F.Cu at (165.2, 61.7)
- added D9: LED1206, LED_SMD:LED_1206_3216Metric, F.Cu at (172.3, 61.7)
- added J1: BAT+, TokeiDigital:Power Pin, B.Cu at (-100.0, 21.0)
- added J2: BAT-, TokeiDigital:Power Pin, B.Cu at (-100.0, 27.0)
- added J5: SPKR+, TokeiDigital:Power Pin, B.Cu at (258.5, 40.5)
- added J6: SPKR-, TokeiDigital:Power Pin, B.Cu at (258.5, 46.5)
- added R1: 1K, TokeiDigital:R_0805, B.Cu at (-107.8, 52.8)
- added R3: 10K, TokeiDigital:R_0805, B.Cu at (-83.5, 106.0)
- added R7: 320R, TokeiDigital:R_0805, B.Cu at (-106.2, 85.5)
- added R8: 3K3, TokeiDigital:R_0805, B.Cu at (-106.2, 89.5)
- added R9: 1K, TokeiDigital:R_0805, B.Cu at (-127.4, 79.4)
- added S1: SWITCH-DPDT, TokeiDigital:SW_DPDT_SMD_MINI, B.Cu at (111.0, 79.5)
- added S10: Push Button, TokeiDigital:Tactile SW SMD, F.Cu at (206.5, 84.7)
- added S11: Push Button, TokeiDigital:Tactile SW SMD, F.Cu at (206.5, 41.0)
- added S12: Push Button, TokeiDigital:Tactile SW SMD, F.Cu at (220.2, 51.9)
- added S13: Push Button, TokeiDigital:Tactile SW SMD, F.Cu at (220.2, 62.8)
- added S14: Push Button, TokeiDigital:Tactile SW SMD, F.Cu at (220.2, 73.7)
- added S15: Push Button, TokeiDigital:Tactile SW SMD, F.Cu at (220.2, 84.7)
- added S16: Push Button, TokeiDigital:Tactile SW SMD, F.Cu at (220.2, 41.0)
- added S17: Push Button, TokeiDigital:Tactile SW SMD, F.Cu at (233.9, 51.9)
- added S18: Push Button, TokeiDigital:Tactile SW SMD, F.Cu at (233.9, 62.8)
- added S19: Push Button, TokeiDigital:Tactile SW SMD, F.Cu at (233.9, 73.7)
- added S2: Push Button, TokeiDigital:Tactile SW SMD, F.Cu at (117.0, 84.7)
- added S20: Push Button, TokeiDigital:Tactile SW SMD, F.Cu at (233.9, 84.7)
- added S21: Push Button, TokeiDigital:Tactile SW SMD, F.Cu at (133.6, 169.0)
- added S22: Push Button, TokeiDigital:Tactile SW SMD, F.Cu at (247.6, 51.9)
- added S23: Push Button, TokeiDigital:Tactile SW SMD, F.Cu at (247.6, 62.8)
- added S24: Push Button, TokeiDigital:Tactile SW SMD, F.Cu at (247.6, 73.7)
- added S25: Push Button, TokeiDigital:Tactile SW SMD, F.Cu at (247.6, 84.7)
- added S26: Push Button, TokeiDigital:Tactile SW SMD, F.Cu at (143.7, 169.0)
- added S3: Push Button, TokeiDigital:Tactile SW SMD, F.Cu at (117.0, 40.0)
- added S4: Push Button, TokeiDigital:Tactile SW SMD, F.Cu at (95.6, 162.3)
- added S5: Push Button, TokeiDigital:Tactile SW SMD, F.Cu at (95.6, 170.7)
- added S6: Push Button, TokeiDigital:Tactile SW SMD, F.Cu at (95.6, 179.0)
- added S7: Push Button, TokeiDigital:Tactile SW SMD, F.Cu at (206.5, 51.9)
- added S8: Push Button, TokeiDigital:Tactile SW SMD, F.Cu at (206.5, 62.8)
- added S9: Push Button, TokeiDigital:Tactile SW SMD, F.Cu at (206.5, 73.7)
- added U1: ~, TokeiDigital:USBC Lipo Charger Module, B.Cu at (109.0, 51.4)
- added U12: DS3502, Package_SO:MSOP-10_3x3mm_P0.5mm, B.Cu at (-114.3, 93.9)
- added U13: PAM8302AAD, Package_SO:MSOP-8_3x3mm_P0.65mm, B.Cu at (-114.3, 98.5)
- added U3: MAX7221xWG, Package_SO:SOIC-24W_7.5x15.4mm_P1.27mm, B.Cu at (-87.6, 92.0)
- BT1, C8, D3, J3, J4, J5, J6, Y1, Y2: moved to B.Cu
- C10: renamed from C9; footprint TokeiDigital:C_0805 -> TokeiDigital:C_1206; moved to B.Cu
- C2: renamed from C1; footprint TokeiDigital:C_0805 -> TokeiDigital:C_1206; moved to B.Cu
- C4: renamed from C2; footprint TokeiDigital:C_0805 -> TokeiDigital:C_1206; moved to B.Cu
- C5: renamed from C3; footprint TokeiDigital:C_0805 -> TokeiDigital:C_1206; moved to B.Cu
- C6: renamed from C4; footprint TokeiDigital:C_0805 -> TokeiDigital:C_1206; moved to B.Cu
- C7: renamed from C5; footprint TokeiDigital:C_0805 -> TokeiDigital:C_1206; moved to B.Cu
- C8: renamed from C6; footprint TokeiDigital:C_0805 -> TokeiDigital:C_1206; moved to B.Cu
- C9: renamed from C7; footprint TokeiDigital:C_0805 -> TokeiDigital:C_1206; moved to B.Cu
- D67: renamed from D1; moved to B.Cu
- D68: renamed from D2; moved to B.Cu
- J3: renamed from J1; footprint TokeiDigital:PIN 1x06 -> Connector_PinSocket_2.54mm:PinSocket_1x06_P2.54mm_Horizontal; moved to B.Cu
- J4: renamed from J2; moved to B.Cu
- R2: renamed from R1; moved to B.Cu
- R4: renamed from R2; moved to B.Cu
- R5: renamed from R3; moved to B.Cu
- R6: renamed from R4; moved to B.Cu
- U10: renamed from U8; footprint TokeiDigital:TQFP-32 -> Package_QFP:TQFP-32_7x7mm_P0.8mm; moved to B.Cu
- U11: renamed from U9; moved to B.Cu
- U2: renamed from U1; moved to B.Cu
- U4: renamed from U2; value Sx39-1xxxxx -> 3191AS
- U5: renamed from U3; value Sx39-1xxxxx -> 3191AS
- U6: renamed from U4; value Sx39-1xxxxx -> 3191AS
- U7: renamed from U5; value Sx39-1xxxxx -> 3191AS
- U8: renamed from U6; value Sx39-1xxxxx -> 3191AS
- U9: renamed from U7; value Sx39-1xxxxx -> 3191AS
- moved J3 184.7 mm to (262.6, 70.2), turned to 180 degrees
- moved U10 181.7 mm to (-85.7, 53.3), turned to 180 degrees
- moved Y1 168.7 mm to (-79.2, 65.1), turned to 180 degrees
- moved D67 168.5 mm to (-79.1, 70.6), turned to 180 degrees
- moved D68 168.5 mm to (-79.1, 74.9), turned to 180 degrees
- moved D3 152.1 mm to (-70.9, 81.1), turned to 180 degrees
- moved C8 150.3 mm to (-70.0, 85.0), turned to 180 degrees
- moved C4 139.3 mm to (-64.5, 38.3), turned to 180 degrees
- moved C5 139.3 mm to (-64.5, 41.3), turned to 180 degrees
- moved C6 139.3 mm to (-64.5, 44.3), turned to 180 degrees
- moved C7 139.3 mm to (-64.5, 47.3), turned to 180 degrees
- moved C8 139.3 mm to (-64.5, 50.3), turned to 180 degrees
- moved C9 139.3 mm to (-64.5, 53.4), turned to 180 degrees
- moved J5 138.3 mm to (-64.0, 82.0), turned to 180 degrees
- moved J6 138.3 mm to (-64.0, 88.0), turned to 180 degrees
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Connections:
- U10 pad 1: /Core/TM1637_CLK -> /BTN_COL1
- U10 pad 10: unconnected-(U8-PD6-Pad10) -> /BTN_COL4
- U10 pad 11: unconnected-(U8-PD7-Pad11) -> /BTN_COL5
- U10 pad 12: /Core/BTNA -> unconnected-(U10-PB0-Pad12)
- U10 pad 13: /Core/BTNB -> /AUDIOPWM
- U10 pad 14: /Core/BTNC -> /BTN_FN
- U10 pad 19: unconnected-(U8-PE2-Pad19) -> /DISP_DATA
- U10 pad 2: /Core/TM1637_CLK -> /BTN_COL2
- U10 pad 23: /Core/TIMED -> /BTN_ROW0
- U10 pad 24: /Core/TIMEC -> /BTN_ROW1
- U10 pad 25: unconnected-(U8-PC2-Pad25) -> /BTN_ROW2
- U10 pad 26: unconnected-(U8-PC3-Pad26) -> /BTN_ROW3
- U10 pad 27: /Core/SDA -> /SDA
- U10 pad 28: /Core/SCL -> /SCL
- U10 pad 3: unconnected-(U8-PE0-Pad3) -> /DISP_!CS
- U10 pad 32: /Core/TM1637_DIO -> /BTN_COL0
- U10 pad 6: unconnected-(U8-PE1-Pad6) -> /DISP_CLK
- U10 pad 9: /Core/WS2812_D -> /BTN_COL3
- U11 pad 5: /rtc/SDA -> /SDA
- U11 pad 6: /rtc/SCL -> /SCL
- U11 pad 7: /rtc/1HZ -> unconnected-(U11-SQW-Pad7)
- U2 pad 1: /Display/DIN -> /DISP_DATA
- U2 pad 10: /Display/C4 -> /Display/C5
- U2 pad 12: /Display/!CS -> /DISP_!CS
- U2 pad 13: /Display/CLK -> /DISP_CLK
- U2 pad 24: unconnected-(U1-DOUT-Pad24) -> /Display/DN1
- U6 pad 10: /Display/A -> /Display/D
- U6 pad 2: /Display/F -> /Display/C
- U6 pad 4: /Display/E -> /Display/B
- U6 pad 5: /Display/D -> /Display/A
- U6 pad 7: /Display/C -> /Display/F
- U6 pad 9: /Display/B -> /Display/E
- U8 pad 10: /Display/A -> /Display/D
- U8 pad 2: /Display/F -> /Display/C
- U8 pad 4: /Display/E -> /Display/B
- U8 pad 5: /Display/D -> /Display/A
- U8 pad 7: /Display/C -> /Display/F
- U8 pad 9: /Display/B -> /Display/E
Routing:
- net (no net): vias 0 -> 4
Other:
- board outline added: 156 x 67 mm
- board text added: "+1"
- board text added: "+10"
- board text added: "+5"
- board text added: "-1"
- board text added: "0"
- board text added: "1"
- board text added: "2"
- board text added: "3"
- board text added: "4"
- board text added: "5"
- board text added: "6"
- board text added: "7"
- board text added: "8"
- board text added: "9"
- board text added: "A"
- board text added: "AD"
- board text added: "B"
- board text added: "C"
- board text added: "D"
- board text added: "DA"
- board text added: "E"
- board text added: "F"
- board text added: "FN"
- board text added: "H"
- board text added: "LR"
- board text added: "M"
- board text added: "MUTE"
- board text added: "NUM"
- board text added: "PRE"
- board text added: "PRG"
- board text added: "S"
- board text added: "SEL"
- board text added: "SS"
- board text added: "T0"
- board text added: "T1"
- board text added: "T2"
- board text added: "T3"
