File: board/TD-TOE01/TD-TOE01.kicad_pcb (KiCad board)
At the start: 2 copper layers, 156 x 67 mm, 146 parts, among them J1 BAT+, J2 BAT-, J3 Pin 1x5, J3 Pin 1x6, J4 AVR-ISP, J4 Pin 1x6, J5 PowerPad, J5 SPKR+, J6 PowerPad, J6 SPKR-, U10 ATmega328PB-QFP, U11 DS1307, U12 DS3502, U13 PAM8302AAD, U2 MAX7221xWG, U3 MAX7221xWG, U4 3191AS, U5 3191AS, U6 3191AS, U7 3191AS, U8 3191AS, U9 3191AS, Y1 16MHz, Y2 32.768KHz

Commit message: OET PCB
Parts:
- removed BT1: CR3032 Holder, TokeiDigital:CR2032 Holder
- removed the C8 at (-70.0, 85.0)
- removed the D3 at (-70.9, 81.1)
- removed the J3 at (-30.5, 104.8)
- removed the J4 at (-25.8, 104.8)
- removed the J5 at (-64.0, 82.0)
- removed the J6 at (-64.0, 88.0)
- removed S21, S26, S4, S5, S6: Push Button, TokeiDigital:Tactile SW SMD
- removed U1: ~, TokeiDigital:USBC Lipo Charger Module
- removed Y2: 32.768KHz, TokeiDigital:Crystal Horizontal
- added C16: 0.33F, TokeiDigital:StarcapSuperCap-HType, B.Cu at (93.4, 91.0)
- added D69: BAT54, Package_TO_SOT_SMD:TSOT-23, B.Cu at (121.7, 99.0)
- added D70: BAT54, Package_TO_SOT_SMD:TSOT-23, B.Cu at (121.8, 106.6)
- added J7: USB-C Receptacle Power Only, TokeiDigital:AMPHENOL_12402012E212A, B.Cu at (73.2, 86.4)
- added J8: BAT+, TokeiDigital:Power Pin, B.Cu at (142.7, 119.2)
- added J9: BAT-, TokeiDigital:Power Pin, B.Cu at (135.9, 119.2)
- added R10: 470R, TokeiDigital:R_0805, B.Cu at (113.9, 100.0)
- added R11: 2K2, TokeiDigital:R_0805, B.Cu at (108.3, 81.0)
- added R12: 5K1, TokeiDigital:R_0805, B.Cu at (108.3, 84.0)
- added R13: 5K1, TokeiDigital:R_0805, B.Cu at (108.3, 86.9)
- added U14: DS3231S, Package_SO:SOIC-16W_7.5x10.3mm_P1.27mm, B.Cu at (118.0, 89.9)
- D1, D67, D68: value 1N5817 -> BAT54; footprint TokeiDigital:D_2010 -> Package_TO_SOT_SMD:TSOT-23
- D2: moved to F.Cu
- R1: value 1K -> 470R
- U11: value DS1307 -> MCP73831-2-OT; footprint TokeiDigital:SOIC-8 -> Package_TO_SOT_SMD:SOT-23-5
- U4, U5, U6, U7, U8, U9: value 3191AS -> Sx39-1xxxxx
- Y1: footprint TokeiDigital:Crystal Vertical -> TokeiDigital:Crystal_SMD_HC49-SD_HandSoldering
- moved R9 340.7 mm to (212.4, 104.5)
- moved R7 318.8 mm to (212.5, 96.3)
- moved R8 318.8 mm to (212.5, 100.3)
- moved U13 315.7 mm to (201.3, 108.8)
- moved U12 315.6 mm to (201.3, 98.7)
- moved C11 290.1 mm to (192.1, 96.5)
- moved C12 290.1 mm to (192.1, 100.6)
- moved C13 290.1 mm to (192.1, 104.7)
- moved C14 290.1 mm to (192.1, 108.7)
- moved C15 290.1 mm to (192.1, 112.8)
- moved C3 285.2 mm to (199.5, 62.2)
- moved U3 284.1 mm to (195.9, 72.6)
- moved R3 278.8 mm to (191.8, 62.0)
- moved D55 274.0 mm to (213.2, 63.3)
- moved D57 273.9 mm to (213.2, 70.4)
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Connections:
- C10 pad 1: GND -> +5V
- C10 pad 2: +5V -> GND
- D1 pad 1: +5V -> Net-(D1-K)
- D1 pad 2: Net-(D1-A) -> unconnected-(D1-NC-Pad2)
- D2 pad 1: GND -> Net-(D2-K)
- D67 pad 1: +5V -> Net-(D67-K)
- D67 pad 2: Net-(D67-A) -> unconnected-(D67-NC-Pad2)
- D68 pad 1: +5V -> Net-(D68-A)
- D68 pad 2: Net-(D68-A) -> unconnected-(D68-NC-Pad2)
- J1 pad 1: Net-(U1-BAT+) -> Net-(U11-V_{BAT})
- J2 pad 1: Net-(U1-BAT-) -> GND
- J3 pad 3: Net-(D67-A) -> Net-(D1-K)
- J4 pad 2: Net-(D68-A) -> Net-(D67-K)
- R1 pad 1: +5V -> Net-(D68-K)
- S1 pad 5: Net-(U1-OUT+) -> Net-(U11-V_{BAT})
- S1 pad 6: Net-(D1-A) -> Net-(D70-K)
- U10 pad 22: unconnected-(U10-PE3-Pad22) -> /RTCINT
- U11 pad 1: Net-(U11-X1) -> Net-(D2-K)
- U11 pad 2: Net-(U11-X2) -> GND
- U11 pad 3: Net-(BT1-+) -> Net-(U11-V_{BAT})
- U11 pad 4: GND -> Net-(D68-K)
- U11 pad 5: /SDA -> Net-(U11-PROG)
Routing:
- net GND: vias 0 -> 6
- net (no net): vias 4 -> 0
Other:
- board text added: "-"
- board text added: "AD/SS"
- board text added: "BAT+"
- board text added: "BAT-"
- board text added: "CHG"
- board text added: "DA/LR"
- board text added: "GND"
- board text added: "L"
- board text added: "T"
- board text added: "Vin"
- board text removed: "LR"
- board text removed: "SS"
