File: board/TD-TOE01/TD-TOE01.kicad_sch (KiCad schematic)
At the start: 25 parts, among them J1 Pin 1x5, J4 Pin 1x6, J5 PowerPad, J6 Pin 1x6, J7 AVR-ISP, J8 PowerPad, U2 DS1307, U3 ATmega328PB-QFP, Y1 16MHz, Y2 32.768KHz

Commit message: OET First steps
Parts:
- removed BT1: CR3032 Holder, TokeiDigital:CR2032 Holder, symbol ClockIt:Battery_Cell
- removed C1, C2: 22p, TokeiDigital:C_0805, symbol ClockIt:C_Small
- removed C3, C4, C5, C6, C7: 100nF, TokeiDigital:C_0805, symbol ClockIt:C_Small
- removed C8: 10uF, TokeiDigital:C_1206, symbol ClockIt:C_Small
- removed D1, D2, D3: 1N5817, TokeiDigital:D_2010, symbol ClockIt:1N5817
- removed J1: Pin 1x5, TokeiDigital:PIN 1x05, symbol ClockIt:Conn_01x05_Socket_1
- removed J4, J6: Pin 1x6, TokeiDigital:PIN 1x06, symbol ClockIt:Conn_01x06_Socket
- removed J5, J8: PowerPad, TokeiDigital:Power Pin, symbol ClockIt:PowerPad
- removed J7: AVR-ISP, TokeiDigital:PIN 2x03, symbol ClockIt:AVR-ISP-6
- removed R1, R2, R3: 10K, TokeiDigital:R_0805, symbol Device:R
- removed U2: DS1307, TokeiDigital:SOIC-8, symbol ClockIt:DS1307
- removed U3: ATmega328PB-QFP, TokeiDigital:TQFP-32, symbol ClockIt:ATmega328PB-QFP
- removed Y1: 16MHz, TokeiDigital:Crystal Vertical, symbol ClockIt:Crystal
- removed Y2: 32.768KHz, TokeiDigital:Crystal Horizontal, symbol ClockIt:Crystal
Connections:
- no-connect marks 8 -> 0
Other:
- added sheet Core (core.kicad_sch)
- added sheet Display (display.kicad_sch)
- added sheet Power (power.kicad_sch)
- added sheet rtc (rtc.kicad_sch)
- note removed: "*1)"
- note removed: "*1) C4 should be omitted if the Arduino bootloader is flashed. This allows for a more reliable reset when the DTR line is toggled. Iterations past REV.A will remove this cap anyway. *2) While PD7 is not connected to the board it is used as an output sending a heartbeat with a 1Hz frequency. This can be used to check the firmware is running. If this pins goes high once every 8s instead it means th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"
- note removed: "*2)"
- note removed: "CTS"
- note removed: "DTR"
- note removed: "GND"
- note removed: "RX"
- note removed: "TX"
- note removed: "VCC"

Commit message: OET schematic
Parts:
- added C1: 10uF, TokeiDigital:C Rect P5.00, symbol TokeiDigital:C_Polarized
- added D1: 1N5817, Diode_THT:D_DO-41_SOD81_P10.16mm_Horizontal, symbol TokeiDigital:1N5817
- added D2: LED1206, LED_SMD:LED_1206_3216Metric, symbol TokeiDigital:LED1206
- added J1: BAT+, TokeiDigital:Power Pin, symbol TokeiDigital:PowerPad
- added J2: BAT-, TokeiDigital:Power Pin, symbol TokeiDigital:PowerPad
- added R1: 1K, TokeiDigital:R_0805, symbol Device:R
- added S1: SWITCH-DPDT, symbol TokeiDigital:SWITCH-DPDT
- added U1: ~, symbol TokeiDigital:LipoCharger
Connections:
- new net: J2.1, U1.3 (BAT-)
- new net: D1.2 (A), S1.5
- new net: D2.2 (A), R1.2
- new net: S1.6, U1.1 (OUT+)
- new net: J1.1, U1.2 (BAT+)
- new net +5V: C1.1, D1.1 (K), R1.1
- new net GND: C1.2, D2.1 (K), U1.4 (OUT-)
- no-connect marks 0 -> 6
Other:
- sheet rtc renamed RTC
- removed sheet Power
- added sheet Audio (audio.kicad_sch)
- added sheet Keyboard (keyboard.kicad_sch)
- sheet Core ports: added BTN_COL0, BTN_COL1, BTN_COL2, BTN_COL3, BTN_COL4, BTN_COL5, BTN_ROW0, BTN_ROW1, BTN_ROW2, BTN_ROW3, BTN_SEL, DISP_!CS, DISP_CLK, DISP_DOUT, PWMOUT, SCL, SDA; removed none
- sheet Display ports: added !CS, CLK, DIN; removed none
- sheet RTC ports: added SCL, SDA; removed none

Commit message: OET
Parts:
- C1: footprint TokeiDigital:C Rect P5.00 -> TokeiDigital:C_1206
- D1: footprint Diode_THT:D_DO-41_SOD81_P10.16mm_Horizontal -> TokeiDigital:D_2010
- S1: footprint (none) -> TokeiDigital:SW_DPDT_SMD_MINI; symbol TokeiDigital:SWITCH-DPDT -> TokeiDigital:SWITCH-DPDT_NO_GND
- U1: footprint (none) -> TokeiDigital:USBC Lipo Charger Module
Connections:
- net at D1.2 (A): now also S1.6; no longer S1.5
- net at U1.1 (OUT+): now also S1.5; no longer S1.6
Other:
- sheet Core ports: added BTN_FN; removed BTN_SEL
- sheet Keyboard ports: added BTN_FN; removed BTN_SEL
Changed lines of the file:
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@@
 		)
 	)
-	(label "BTN_SEL"
+	(label "BTN_FN"
 		(at 172.72 57.15 0)
 		(effects
@@
 		)
 	)
-	(label "BTN_SEL"
+	(label "BTN_FN"
 		(at 95.25 25.4 180)
 		(effects
@@
 			)
 		)
-		(property "Footprint" "Diode_THT:D_DO-41_SOD81_P10.16mm_Horizontal"
+		(property "Footprint" "TokeiDigital:D_2010"
 			(at 92.71 116.205 0)
 			(effects
@@
 			)
 		)
-		(property "Footprint" ""
+		(property "Footprint" "TokeiDigital:USBC Lipo Charger Module"
 			(at 48.26 115.57 0)
 			(effects
@@
 			)
 		)
-		(property "Footprint" "TokeiDigital:C Rect P5.00"
+		(property "Footprint" "TokeiDigital:C_1206"
 			(at 107.6452 130.81 0)
 			(effects
@@
 	)
 	(symbol
-		(lib_id "TokeiDigital:SWITCH-DPDT")
+		(lib_id "TokeiDigital:SWITCH-DPDT_NO_GND")
 		(at 78.74 113.03 0)
 		(unit 1)
@@
 			)
 		)
-		(property "Footprint" ""
+		(property "Footprint" "TokeiDigital:SW_DPDT_SMD_MINI"
 			(at 78.74 101.6 0)
 			(effects
@@
 			)
 		)
-		(pin "9"
-		)
 		(pin "2"
 		)
@@
 		(pin "5"
 		)
-		(pin "7"
+		(pin "4"
 		)
 		(pin "1"
 		)
 		(pin "3"
-		)
-		(pin "8"
 		)
 		(instances
@@
 			)
 		)
-		(pin "BTN_SEL" output
+		(pin "BTN_FN" output
 			(at 185.42 57.15 180)
 			(effects
@@
 			)
 		)
-		(pin "BTN_SEL" input
+		(pin "BTN_FN" input
 			(at 83.82 25.4 0)
 			(effects
