File: board/TD-TOE01/TD-TOE01.kicad_sch (KiCad schematic)
At the start: 8 parts, among them J1 BAT+, J2 BAT-

Commit message: OET PCB
Parts:
- removed D1: 1N5817, TokeiDigital:D_2010, symbol TokeiDigital:1N5817
- removed U1: ~, TokeiDigital:USBC Lipo Charger Module, symbol TokeiDigital:LipoCharger
- added D68, D70: BAT54, Package_TO_SOT_SMD:TSOT-23, symbol TokeiDigital:BAT54
- added J7: USB-C Receptacle Power Only, TokeiDigital:AMPHENOL_12402012E212A, symbol TokeiDigital:USB-C Receptacle Power Only
- added J8: BAT+, TokeiDigital:Power Pin, symbol TokeiDigital:PowerPad
- added J9: BAT-, TokeiDigital:Power Pin, symbol TokeiDigital:PowerPad
- added R11: 2K2, TokeiDigital:R_0805, symbol Device:R
- added R12, R13: 5K1, TokeiDigital:R_0805, symbol Device:R
- added U11: MCP73831-2-OT, Package_TO_SOT_SMD:SOT-23-5, symbol TokeiDigital:MCP73831-2-OT
- R1: value 1K -> 470R
Connections:
- net +5V: now also D70.3 (K); no longer R1.1
- net GND: now also J2.1, J7.GND, J7.SHL (SHIELD), J9.1, R11.2, R12.2, R13.2, U11.2 (V_{SS}); no longer D2.1 (K)
- net at S1.6: now also D70.1 (A)
- net at S1.5: now also J1.1, U11.3 (V_{BAT})
- new net: D2.1 (K), U11.1 (STAT)
- new net: D68.3 (K), J7.VBUS, R1.1, U11.4 (V_{DD})
- new net: R11.1, U11.5 (PROG)
- new net: D68.1 (A), J8.1
- new net: J7.CC1, R13.1
- new net: J7.CC2, R12.1
- no-connect marks 6 -> 4
Other:
- sheet Core ports: added RTCINT; removed none
- sheet RTC ports: added INT; removed none
- note added: "+"
- note added: "ICharge=450mA"
- note added: "LiPo Battery"
- note added: "Vin"
- moved on the sheet: C1, D2, J1, J2, R1, S1
