File: board/TD-TOE01/audio.kicad_sch (KiCad schematic)
At the start: 12 parts, among them J5 SPKR+, J6 SPKR-, U12 DS3502, U13 PAM8302AAD

Commit message: OET
Parts:
- C11, C12, C13, C14, C15: footprint TokeiDigital:C Rect P5.00 -> TokeiDigital:C_1206
- J5, J6: footprint (none) -> TokeiDigital:Power Pin
- R7, R8: footprint TokeiDigital:R-Axial -> TokeiDigital:R_0805
- R9: footprint (none) -> TokeiDigital:R_0805
Changed lines of the file:
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@@
 			)
 		)
-		(property "Footprint" "TokeiDigital:C Rect P5.00"
+		(property "Footprint" "TokeiDigital:C_1206"
 			(at 127 66.04 0)
 			(effects
@@
 			)
 		)
-		(property "Footprint" "TokeiDigital:C Rect P5.00"
+		(property "Footprint" "TokeiDigital:C_1206"
 			(at 114.3 66.04 0)
 			(effects
@@
 			)
 		)
-		(property "Footprint" "TokeiDigital:R-Axial"
+		(property "Footprint" "TokeiDigital:R_0805"
 			(at 107.95 62.23 0)
 			(effects
@@
 			)
 		)
-		(property "Footprint" "TokeiDigital:R-Axial"
+		(property "Footprint" "TokeiDigital:R_0805"
 			(at 121.92 62.23 0)
 			(effects
@@
 			)
 		)
-		(property "Footprint" "TokeiDigital:C Rect P5.00"
+		(property "Footprint" "TokeiDigital:C_1206"
 			(at 180.34 104.4448 0)
 			(effects
@@
 			)
 		)
-		(property "Footprint" "TokeiDigital:C Rect P5.00"
+		(property "Footprint" "TokeiDigital:C_1206"
 			(at 101.6 96.52 0)
 			(effects
@@
 		(on_board yes)
 		(dnp no)
-		(fields_autoplaced yes)
 		(property "Reference" "R9"
-			(at 163.83 99.06 90)
+			(at 164.084 107.95 90)
 			(effects
 				(font
@@
 		)
 		(property "Value" "1K"
-			(at 163.83 101.6 90)
-			(effects
-				(font
-					(size 1.27 1.27)
-				)
-			)
-		)
-		(property "Footprint" ""
+			(at 163.576 102.87 90)
+			(effects
+				(font
+					(size 1.27 1.27)
+				)
+			)
+		)
+		(property "Footprint" "TokeiDigital:R_0805"
 			(at 163.83 107.188 90)
 			(effects
@@
 			)
 		)
-		(property "Footprint" "TokeiDigital:C Rect P5.00"
+		(property "Footprint" "TokeiDigital:C_1206"
 			(at 183.1848 91.44 0)
 			(effects
@@
 			)
 		)
-		(property "Footprint" ""
+		(property "Footprint" "TokeiDigital:Power Pin"
 			(at 215.9 115.57 0)
 			(effects
@@
 			)
 		)
-		(property "Footprint" ""
+		(property "Footprint" "TokeiDigital:Power Pin"
 			(at 215.9 110.49 0)
 			(effects
