File: board/TD-TOE01/core.kicad_sch (KiCad schematic)
At the start: 17 parts, among them J1 Pin 1x6, J2 AVR-ISP, J3 Pin 1x5, J4 Pin 1x6, U8 ATmega328PB-QFP, Y1 16MHz

Commit message: OET schematic
Parts:
- removed J3: Pin 1x5, TokeiDigital:PIN 1x05, symbol ClockIt:Conn_01x05_Socket_1
- removed J4: Pin 1x6, TokeiDigital:PIN 1x06, symbol ClockIt:Conn_01x06_Socket
- C4: renamed from C2; footprint TokeiDigital:C_0805 -> TokeiDigital:C Rect P5.00; symbol ClockIt:C_Small -> TokeiDigital:C_Small
- C5: renamed from C3; footprint TokeiDigital:C_0805 -> TokeiDigital:C Rect P5.00; symbol ClockIt:C_Small -> TokeiDigital:C_Small
- C6: renamed from C4; footprint TokeiDigital:C_0805 -> TokeiDigital:C Rect P5.00; symbol ClockIt:C_Small -> TokeiDigital:C_Small
- C7: renamed from C5; footprint TokeiDigital:C_0805 -> TokeiDigital:C Rect P5.00; symbol ClockIt:C_Small -> TokeiDigital:C_Small
- C8: renamed from C6; footprint TokeiDigital:C_0805 -> TokeiDigital:C Rect P5.00; symbol ClockIt:C_Small -> TokeiDigital:C_Small
- C9: renamed from C7; footprint TokeiDigital:C_0805 -> TokeiDigital:C Rect P5.00; symbol ClockIt:C_Small -> TokeiDigital:C_Small
- D67: renamed from D1; footprint TokeiDigital:D_2010 -> Diode_THT:D_DO-41_SOD81_P10.16mm_Horizontal; symbol ClockIt:1N5817 -> TokeiDigital:1N5817
- D68: renamed from D2; footprint TokeiDigital:D_2010 -> Diode_THT:D_DO-41_SOD81_P10.16mm_Horizontal; symbol ClockIt:1N5817 -> TokeiDigital:1N5817
- J3: renamed from J1; footprint TokeiDigital:PIN 1x06 -> Connector_PinSocket_2.54mm:PinSocket_1x06_P2.54mm_Horizontal; symbol ClockIt:Conn_01x06_Socket -> TokeiDigital:Conn_01x06_Socket
- J4: renamed from J2; symbol ClockIt:AVR-ISP-6 -> TokeiDigital:AVR-ISP-6
- U10: renamed from U8; footprint TokeiDigital:TQFP-32 -> Package_QFP:TQFP-32_7x7mm_P0.8mm; symbol ClockIt:ATmega328PB-QFP -> TokeiDigital:ATmega328PB-QFP
- Y1: symbol ClockIt:Crystal -> TokeiDigital:Crystal
- renumbered R2 to R4, R3 to R5, R4 to R6
Connections:
- net BTN_COL4: now reaches U10.10 (PD6)
- net BTN_COL5: now reaches U10.11 (PD7)
- net DISP_DOUT: now reaches U10.19 (PE2)
- net BTN_ROW2: now reaches U10.25 (PC2)
- net BTN_ROW3: now reaches U10.26 (PC3)
- net DISP_!CS: now reaches U10.3 (PE0)
- net DISP_CLK: now reaches U10.6 (PE1)
- net BTNA: no longer names the net of U10.12 (PB0)
- net BTNB renamed PWMOUT
- net BTNC renamed BTN_SEL
- net TIMEC renamed BTN_ROW1
- net TIMED renamed BTN_ROW0
- net TM1637_CLK renamed BTN_COL1
- net BTN_COL1: no longer U10.2 (PD4)
- net TM1637_DIO renamed BTN_COL0
- net WS2812_D renamed BTN_COL3
- new net BTN_COL2: U10.2 (PD4)
- no-connect marks 8 -> 2
Other:
- note removed: "*1)"
- note removed: "*1) C4 should be omitted if the Arduino bootloader is flashed. This allows for a more reliable reset when the DTR line is toggled. Iterations past REV.A will remove this cap anyway. *2) While PD7 is not connected to the board it is used as an output sending a heartbeat with a 1Hz frequency. This can be used to check the firmware is running. If this pins goes high once every 8s instead it means th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"
- note removed: "*2)"
- moved on the sheet: C4, C5, C6, C7, C8, C9, D67, D68, J3, J4, R4, R5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

Commit message: OET
Parts:
- C4, C5, C6, C7, C8, C9: footprint TokeiDigital:C Rect P5.00 -> TokeiDigital:C_1206
- D67, D68: footprint Diode_THT:D_DO-41_SOD81_P10.16mm_Horizontal -> TokeiDigital:D_2010
Connections:
- net BTN_SEL renamed BTN_FN
Changed lines of the file:
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@@
 		)
 	)
-	(hierarchical_label "BTN_SEL"
+	(hierarchical_label "BTN_FN"
 		(shape input)
 		(at 151.13 63.5 0)
@@
 			)
 		)
-		(property "Footprint" "TokeiDigital:C Rect P5.00"
+		(property "Footprint" "TokeiDigital:C_1206"
 			(at 128.27 135.89 0)
 			(effects
@@
 			)
 		)
-		(property "Footprint" "TokeiDigital:C Rect P5.00"
+		(property "Footprint" "TokeiDigital:C_1206"
 			(at 133.35 48.26 0)
 			(effects
@@
 			)
 		)
-		(property "Footprint" "TokeiDigital:C Rect P5.00"
+		(property "Footprint" "TokeiDigital:C_1206"
 			(at 101.6 73.66 0)
 			(effects
@@
 			)
 		)
-		(property "Footprint" "Diode_THT:D_DO-41_SOD81_P10.16mm_Horizontal"
+		(property "Footprint" "TokeiDigital:D_2010"
 			(at 78.105 80.01 0)
 			(effects
@@
 			)
 		)
-		(property "Footprint" "TokeiDigital:C Rect P5.00"
+		(property "Footprint" "TokeiDigital:C_1206"
 			(at 93.98 73.66 0)
 			(effects
@@
 			)
 		)
-		(property "Footprint" "TokeiDigital:C Rect P5.00"
+		(property "Footprint" "TokeiDigital:C_1206"
 			(at 107.95 62.23 0)
 			(effects
@@
 			)
 		)
-		(property "Footprint" "TokeiDigital:C Rect P5.00"
+		(property "Footprint" "TokeiDigital:C_1206"
 			(at 118.11 135.89 0)
 			(effects
@@
 			)
 		)
-		(property "Footprint" "Diode_THT:D_DO-41_SOD81_P10.16mm_Horizontal"
+		(property "Footprint" "TokeiDigital:D_2010"
 			(at 182.245 53.34 0)
 			(effects
