File: board/TD-TOE01/core.kicad_sch (KiCad schematic)
At the start: 15 parts, among them J3 Pin 1x6, J4 AVR-ISP, U10 ATmega328PB-QFP, Y1 16MHz

Commit message: OET PCB
Parts:
- removed D67, D68: 1N5817, TokeiDigital:D_2010, symbol TokeiDigital:1N5817
- added D1, D67: BAT54, Package_TO_SOT_SMD:TSOT-23, symbol TokeiDigital:BAT54
- Y1: footprint TokeiDigital:Crystal Vertical -> TokeiDigital:Crystal_SMD_HC49-SD_HandSoldering
Connections:
- net +5V: now also D1.3 (K), D67.3 (K)
- net RTCINT: now reaches U10.22 (PE3)
- net at J3.3 (Pin_3): now also D1.1 (A)
- net at J4.2 (VCC): now also D67.1 (A)
- no-connect marks 2 -> 1
Changed lines of the file:
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@@
 		(at 143.51 58.42)
 	)
-	(no_connect
-		(at 111.76 111.76)
-	)
 	(wire
 		(pts
@@
 	(wire
 		(pts
+			(xy 104.14 111.76) (xy 113.03 111.76)
+		)
+		(stroke
+			(width 0)
+			(type default)
+		)
+	)
+	(wire
+		(pts
 			(xy 104.14 109.22) (xy 113.03 109.22)
 		)
@@
 		(pts
 			(xy 177.8 46.99) (xy 177.8 49.53)
-		)
-		(stroke
-			(width 0)
-			(type default)
-		)
-	)
-	(wire
-		(pts
-			(xy 111.76 111.76) (xy 113.03 111.76)
 		)
 		(stroke
@@
 			)
 			(justify left)
+		)
+	)
+	(hierarchical_label "RTCINT"
+		(shape input)
+		(at 104.14 111.76 180)
+		(effects
+			(font
+				(size 1.27 1.27)
+			)
+			(justify right)
 		)
 	)
@@
 	)
 	(symbol
+		(lib_id "TokeiDigital:BAT54")
+		(at 177.8 53.34 270)
+		(unit 1)
+		(exclude_from_sim no)
+		(in_bom yes)
+		(on_board yes)
+		(dnp no)
+		(fields_autoplaced yes)
+		(property "Reference" "D67"
+			(at 180.34 51.7524 90)
+			(effects
+				(font
+					(size 1.27 1.27)
+				)
+				(justify left)
+			)
+		)
+		(property "Value" "BAT54"
+			(at 180.34 54.2924 90)
+			(effects
+				(font
+					(size 1.27 1.27)
+				)
+				(justify left)
+			)
+		)
+		(property "Footprint" "Package_TO_SOT_SMD:TSOT-23"
+			(at 173.355 53.34 0)
+			(effects
+				(font
+					(size 1.27 1.27)
+				)
+				(hide yes)
+			)
+		)
+		(property "Datasheet" "https://assets.nexperia.com/documents/data-sheet/BAT54J.pdf"
+			(at 177.8 53.34 0)
+			(effects
+				(font
+					(size 1.27 1.27)
+				)
+				(hide yes)
+			)
+		)
+		(property "Description" "30V 200mA Schottky diode, SOD-323F"
+			(at 177.8 53.34 0)
+			(effects
+				(font
+					(size 1.27 1.27)
+				)
+				(hide yes)
+			)
+		)
+		(pin "1"
+		)
+		(pin "2"
+		)
+		(pin "3"
+		)
+		(instances
+			(project "TD-TOE01"
+				(path "/bdccfd91-2131-490c-a91d-88ce438b2c4c/51dbbb27-08dd-4268-ae44-9a0f21ab928b"
+					(reference "D67")
+					(unit 1)
+				)
+			)
+		)
+	)
+	(symbol
 		(lib_name "GND_1")
 		(lib_id "power:GND")
@@
 	)
 	(symbol
-		(lib_id "TokeiDigital:1N5817")
-		(at 82.55 80.01 270)
-		(unit 1)
-		(exclude_from_sim no)
-		(in_bom yes)
-		(on_board yes)
-		(dnp no)
-		(property "Reference" "D67"
-			(at 86.36 82.55 90)
-			(effects
-				(font
-					(size 1.27 1.27)
-				)
-				(justify right)
-			)
-		)
-		(property "Value" "1N5817"
-			(at 80.01 80.01 90)
-			(effects
-				(font
-					(size 1.27 1.27)
-				)
-				(justify right)
-			)
-		)
-		(property "Footprint" "TokeiDigital:D_2010"
-			(at 78.105 80.01 0)
-			(effects
-				(font
-					(size 1.27 1.27)
-				)
-				(hide yes)
-			)
-		)
-		(property "Datasheet" "http://www.vishay.com/docs/88525/1n5817.pdf"
-			(at 82.55 80.01 0)
-			(effects
-				(font
-					(size 1.27 1.27)
-				)
-				(hide yes)
-			)
-		)
-		(property "Description" "20V 1A Schottky Barrier Rectifier Diode, DO-41"
-			(at 82.55 80.01 0)
-			(effects
-				(font
-					(size 1.27 1.27)
-				)
-				(hide yes)
-			)
-		)
-		(property "Buy" "https://www.aliexpress.com/item/1005001552094086.html?spm=a2g0o.productlist.main.1.2e94WwbYWwbY5g&algo_pvid=c0be6ba8-0814-418b-8f57-5b462f90716d&algo_exp_id=c0be6ba8-0814-418b-8f57-5b462f90716d-0&pdp_npi=4%40dis%21EUR%210.32%210.32%21%21%210.33%21%21%40211b815c16974702438423181e37e4%2112000016564939110%21sea%21PL%212225465097%21&curPageLogUid=UOM2CuyYhq8v"
-			(at 82.55 80.01 0)
-			(effects
-				(font
-					(size 1.27 1.27)
-				)
-				(hide yes)
-			)
-		)
-		(property "Price" "0.015"
-			(at 82.55 80.01 0)
-			(effects
-				(font
-					(size 1.27 1.27)
-				)
-				(hide yes)
-			)
-		)
-		(pin "1"
-		)
-		(pin "2"
-		)
-		(instances
-			(project "TD-TOE01"
-				(path "/bdccfd91-2131-490c-a91d-88ce438b2c4c/51dbbb27-08dd-4268-ae44-9a0f21ab928b"
-					(reference "D67")
-					(unit 1)
-				)
-			)
-		)
-	)
-	(symbol
 		(lib_id "TokeiDigital:AVR-ISP-6")
 		(at 179.07 71.12 0)
@@
 	)
 	(symbol
+		(lib_id "TokeiDigital:BAT54")
+		(at 82.55 80.01 270)
+		(unit 1)
+		(exclude_from_sim no)
+		(in_bom yes)
+		(on_board yes)
+		(dnp no)
+		(fields_autoplaced yes)
+		(property "Reference" "D1"
+			(at 85.09 78.4224 90)
+			(effects
+				(font
+					(size 1.27 1.27)
+				)
+				(justify left)
+			)
+		)
+		(property "Value" "BAT54"
+			(at 85.09 80.9624 90)
+			(effects
+				(font
+					(size 1.27 1.27)
+				)
+				(justify left)
+			)
+		)
+		(property "Footprint" "Package_TO_SOT_SMD:TSOT-23"
+			(at 78.105 80.01 0)
+			(effects
+				(font
+					(size 1.27 1.27)
+				)
+				(hide yes)
+			)
+		)
+		(property "Datasheet" "https://assets.nexperia.com/documents/data-sheet/BAT54J.pdf"
+			(at 82.55 80.01 0)
+			(effects
+				(font
+					(size 1.27 1.27)
+				)
+				(hide yes)
+			)
+		)
+		(property "Description" "30V 200mA Schottky diode, SOD-323F"
+			(at 82.55 80.01 0)
+			(effects
+				(font
+					(size 1.27 1.27)
+				)
+				(hide yes)
+			)
+		)
+		(pin "1"
+		)
+		(pin "2"
+		)
+		(pin "3"
+		)
+		(instances
+			(project "TD-TOE01"
+				(path "/bdccfd91-2131-490c-a91d-88ce438b2c4c/51dbbb27-08dd-4268-ae44-9a0f21ab928b"
+					(reference "D1")
+					(unit 1)
+				)
+			)
+		)
+	)
+	(symbol
 		(lib_id "TokeiDigital:Crystal")
 		(at 123.19 130.81 0)
@@
 			)
 		)
-		(property "Footprint" "TokeiDigital:Crystal Vertical"
+		(property "Footprint" "TokeiDigital:Crystal_SMD_HC49-SD_HandSoldering"
 			(at 123.19 130.81 0)
 			(effects
@@
 					(unit 1)
 				)
-			)
-		)
-	)
-	(symbol
-		(lib_id "TokeiDigital:1N5817")
-		(at 177.8 53.34 90)
-		(mirror x)
-		(unit 1)
-		(exclude_from_sim no)
-		(in_bom yes)
-		(on_board yes)
-		(dnp no)
-		(property "Reference" "D68"
-			(at 172.72 55.88 90)
-			(effects
-				(font
-					(size 1.27 1.27)
-				)
-				(justify right)
-			)
-		)
-		(property "Value" "1N5817"
-			(at 168.91 53.34 90)
-			(effects
-				(font
-					(size 1.27 1.27)
-				)
-				(justify right)
-			)
-		)
-		(property "Footprint" "TokeiDigital:D_2010"
-			(at 182.245 53.34 0)
-			(effects
-				(font
-					(size 1.27 1.27)
-				)
-				(hide yes)
-			)
-		)
-		(property "Datasheet" "http://www.vishay.com/docs/88525/1n5817.pdf"
-			(at 177.8 53.34 0)
-			(effects
-				(font
-					(size 1.27 1.27)
-				)
-				(hide yes)
-			)
-		)
-		(property "Description" "20V 1A Schottky Barrier Rectifier Diode, DO-41"
-			(at 177.8 53.34 0)
-			(effects
-				(font
-					(size 1.27 1.27)
-				)
-				(hide yes)
-			)
-		)
-		(property "Buy" "https://www.aliexpress.com/item/1005001552094086.html?spm=a2g0o.productlist.main.1.2e94WwbYWwbY5g&algo_pvid=c0be6ba8-0814-418b-8f57-5b462f90716d&algo_exp_id=c0be6ba8-0814-418b-8f57-5b462f90716d-0&pdp_npi=4%40dis%21EUR%210.32%210.32%21%21%210.33%21%21%40211b815c16974702438423181e37e4%2112000016564939110%21sea%21PL%212225465097%21&curPageLogUid=UOM2CuyYhq8v"
-			(at 177.8 53.34 0)
-			(effects
-				(font
-					(size 1.27 1.27)
-				)
-				(hide yes)
-			)
-		)
-		(property "Price" "0.015"
-			(at 177.8 53.34 0)
-			(effects
-				(font
-					(size 1.27 1.27)
-				)
-				(hide yes)
-			)
-		)
-		(pin "1"
-		)
-		(pin "2"
-		)
-		(instances
-			(project "TD-TOE01"
-				(path "/bdccfd91-2131-490c-a91d-88ce438b2c4c/51dbbb27-08dd-4268-ae44-9a0f21ab928b"
-					(reference "D68")
-					(unit 1)
-				)
