File: board/TD-TOE01/display.kicad_sch (KiCad schematic)
At the start: 25 parts, among them U1 MAX7221xWG, U2 3191AS, U3 3191AS, U4 3191AS, U5 3191AS, U6 3191AS, U7 3191AS

Commit message: OET schematic
Parts:
- added C3: 100nF, TokeiDigital:C Rect P5.00, symbol TokeiDigital:C_Small
- added D20, D21, D22, D23, D24, D25, D26, D27, D28, D29, D30, D31, D32, D33, D34, D35, D36, D37, D38, D39, D40, D41, D42, D43, D44, D45, D46, D47, D48, D49, D5, D50, D51, D52, D53, D54, D55, D56, D57, D58, D59, D60, D61, D62, D63, D64, D65, D66: LED1206, LED_SMD:LED_1206_3216Metric, symbol TokeiDigital:LED1206
- added R3: 10K, TokeiDigital:R_0805, symbol Device:R
- added U3: MAX7221xWG, Package_SO:SOIC-24W_7.5x15.4mm_P1.27mm, symbol TokeiDigital:MAX7221xWG
- C2: renamed from C1; footprint TokeiDigital:C_0805 -> TokeiDigital:C Rect P5.00; symbol ClockIt:C_Small -> TokeiDigital:C_Small
- renumbered D5 to D3, R1 to R2, U1 to U2, U2 to U4, U3 to U5, U4 to U6, U5 to U7, U6 to U8, U7 to U9
Connections:
- net !CS: now also U3.12 (~{CS})
- net +5V: now also C3.2, R3.1, U3.19 (V+)
- net A: now also U6.5 (D), U8.5 (D); no longer D12.2 (A), D3.2 (A), U6.10 (A), U8.10 (A)
- net B: now also U6.4 (E), U8.4 (E); no longer D13.2 (A), D6.2 (A), U6.9 (B), U8.9 (B)
- net C: now also U6.2 (F), U8.2 (F); no longer D14.2 (A), D4.2 (A), U6.7 (C), U8.7 (C)
- net C4: no longer U2.10 (DIG_5), U2.8 (DIG_7)
- net C5: now also U2.10 (DIG_5); no longer U2.5 (DIG_6)
- net CLK: now also U3.13 (CLK)
- net D: now also U6.10 (A), U8.10 (A); no longer D11.2 (A), D15.2 (A), U6.5 (D), U8.5 (D)
- net DP: no longer D10.2 (A), D19.2 (A)
- net E: now also U6.9 (B), U8.9 (B); no longer D16.2 (A), D7.2 (A), U6.4 (E), U8.4 (E)
- net F: now also U6.7 (C), U8.7 (C); no longer D17.2 (A), D8.2 (A), U6.2 (F), U8.2 (F)
- net G: no longer D18.2 (A), D9.2 (A)
- net GND: now also C3.1, U3.4 (GND), U3.9 (GND)
- net DN1: now reaches U2.24 (DOUT)
- net DN1: now also U3.1 (DIN)
- net C6 renamed LK0
- net LK0: now also D5.1 (K), U3.2 (DIG_0); no longer D11.1 (K)
- net C7 renamed LK4
- net LK4: now also D11.1 (K), U3.3 (DIG_4); no longer D19.1 (K)
- new net: R3.2, U3.18 (ISET)
- new net LA0: D11.2 (A), D19.2 (A), D27.2 (A), D3.2 (A), D35.2 (A), D43.2 (A), D51.2 (A), D59.2 (A), U3.14 (SEG_A)
- new net LA1: D12.2 (A), D20.2 (A), D28.2 (A), D36.2 (A), D4.2 (A), D44.2 (A), D52.2 (A), D60.2 (A), U3.16 (SEG_B)
- new net LA2: D13.2 (A), D21.2 (A), D29.2 (A), D37.2 (A), D45.2 (A), D5.2 (A), D53.2 (A), D61.2 (A), U3.20 (SEG_C)
- new net LA3: D14.2 (A), D22.2 (A), D30.2 (A), D38.2 (A), D46.2 (A), D54.2 (A), D6.2 (A), D62.2 (A), U3.23 (SEG_D)
- new net LA4: D15.2 (A), D23.2 (A), D31.2 (A), D39.2 (A), D47.2 (A), D55.2 (A), D63.2 (A), D7.2 (A), U3.21 (SEG_E)
- new net LA5: D16.2 (A), D24.2 (A), D32.2 (A), D40.2 (A), D48.2 (A), D56.2 (A), D64.2 (A), D8.2 (A), U3.15 (SEG_F)
- new net LA6: D17.2 (A), D25.2 (A), D33.2 (A), D41.2 (A), D49.2 (A), D57.2 (A), D65.2 (A), D9.2 (A), U3.17 (SEG_G)
- new net LA7: D10.2 (A), D18.2 (A), D26.2 (A), D34.2 (A), D42.2 (A), D50.2 (A), D58.2 (A), D66.2 (A), U3.22 (SEG_DP)
- new net LK1: D19.1 (K), D20.1 (K), D21.1 (K), D22.1 (K), D23.1 (K), D24.1 (K), D25.1 (K), D26.1 (K), U3.11 (DIG_1)
- new net LK2: D35.1 (K), D36.1 (K), D37.1 (K), D38.1 (K), D39.1 (K), D40.1 (K), D41.1 (K), D42.1 (K), U3.6 (DIG_2)
- new net LK3: D51.1 (K), D52.1 (K), D53.1 (K), D54.1 (K), D55.1 (K), D56.1 (K), D57.1 (K), D58.1 (K), U3.7 (DIG_3)
- new net LK5: D27.1 (K), D28.1 (K), D29.1 (K), D30.1 (K), D31.1 (K), D32.1 (K), D33.1 (K), D34.1 (K), U3.10 (DIG_5)
- new net LK6: D43.1 (K), D44.1 (K), D45.1 (K), D46.1 (K), D47.1 (K), D48.1 (K), D49.1 (K), D50.1 (K), U3.5 (DIG_6)
- new net LK7: D59.1 (K), D60.1 (K), D61.1 (K), D62.1 (K), D63.1 (K), D64.1 (K), D65.1 (K), D66.1 (K), U3.8 (DIG_7)
- no-connect marks 1 -> 3
Other:
- note added: "NOTE: the minutes and seconds decades displays are flipped on the PCB with the DP to the top left to create a slant semicolon. For this reason segments are not mapped A->A but A->D etc. so that from software perspective all digits work the same. Pay attention to pin1 position on the PCB when assembling."
- note added: "Pay attention to PCB markings this is assembled upside down."
- moved on the sheet: D3, U4, U5, U6, U7, U8, U9

Commit message: OET
Parts:
- C2, C3: footprint TokeiDigital:C Rect P5.00 -> TokeiDigital:C_1206
Changed lines of the file:
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@@
 			)
 		)
-		(property "Footprint" "TokeiDigital:C Rect P5.00"
+		(property "Footprint" "TokeiDigital:C_1206"
 			(at 57.15 109.22 0)
 			(effects
@@
 			)
 		)
-		(property "Footprint" "TokeiDigital:C Rect P5.00"
+		(property "Footprint" "TokeiDigital:C_1206"
 			(at 57.15 35.56 0)
 			(effects
