File: board/TD-TOE01/keyboard.kicad_sch (KiCad schematic)
At the start: 25 parts

Commit message: OET
Connections:
- net BTN_SEL renamed BTN_FN
Changed lines of the file:
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@@
 		)
 	)
-	(hierarchical_label "BTN_SEL"
+	(hierarchical_label "BTN_FN"
 		(shape output)
 		(at 33.02 26.67 180)
