File: board/TD-TOE01/keyboard.kicad_sch (KiCad schematic)
At the start: 25 parts

Commit message: OET PCB
Parts:
- removed S21, S26, S4, S5, S6: Push Button, TokeiDigital:Tactile SW SMD, symbol TokeiDigital:SW_Push
Connections:
- no-connect marks 0 -> 5
